File: CAN_BUS/CAN_BUS.kicad_sch (KiCad schematic)
At the start: 11 parts, among them J1 Conn_01x04_Pin, J2 Conn_01x04_Pin, J3 JST VH B2P-VH-FB-B, J4 JST XH B2B-XH-A, U1 TS12A4514DBVR

Commit message: Add files via upload
Parts:
- removed D2: UCLAMP1071P.TNT, UCLAMP1071P.TNT:DIO_UCLAMP1071P.TNT, symbol Device:D_Zener
- added C3, C4, C5, C6, C7, C8, C9: 0.1uF, Capacitor_SMD:C_1812_4532Metric_Pad1.57x3.40mm_HandSolder, symbol Device:C
- added CR1, CR3, CR4, CR5, CR6: ESD2CAN36DBZRQ1, SOT-23-3_DBZ_TEX, symbol ESD2CAN36-Q1:ESD2CAN36DBZRQ1
- added D1, D3, D4, D5, D6, D7: UCLAMP1071P.TNT, UCLAMP1071P.TNT:DIO_UCLAMP1071P.TNT, symbol UCLAMP1071P.TNT:UCLAMP1071P.TNT
- added J10, J11, J12, J5, J7, J9: Conn_01x04, symbol Connector_Generic:Conn_01x04
- added J13, J14, J23, J26: Conn_01x04, Connector_JST:JST_GH_BM04B-GHS-TBT_1x04-1MP_P1.25mm_Vertical, symbol Connector_Generic:Conn_01x04
- added J15, J16, J24, J25: Conn_01x04_Pin, Connector_JST:JST_GH_BM04B-GHS-TBT_1x04-1MP_P1.25mm_Vertical, symbol Connector:Conn_01x04_Pin
- added J17, J18: JST XH B2B-XH-A, Connector_JST:JST_XH_B2B-XH-A_1x02_P2.50mm_Vertical, symbol Connector:Conn_01x02_Pin
- added J6, J8: JST VH B2P-VH-FB-B, Connector_JST:JST_VH_B2P-VH-FB-B_1x02_P3.96mm_Vertical, symbol Connector:Conn_01x02_Pin
- added R10, R11, R17, R18, R21, R24, R25, R29, R30, R33, R34, R8: 120R, symbol Device:R
- added R12, R19, R20, R22, R23, R31, R32, R7: 10kR, Resistor_SMD:R_1812_4532Metric_Pad1.30x3.40mm_HandSolder, symbol Device:R
- added R13, R9: R, symbol Device:R
- added R14, R16: 10kR, symbol Device:R
- added R15, R5: 120R, Resistor_SMD:R_1812_4532Metric_Pad1.30x3.40mm_HandSolder, symbol Device:R
- added SW1, SW3, SW4, SW5, SW6: SW_MEC_5G, symbol Switch:SW_MEC_5G
- added U2, U4, U5, U6: TS12A4514DBVR, TS12A4514:DBV5, symbol TS12A4514:TS12A4514DBVR
- C1: footprint Capacitor_SMD:C_1206_3216Metric_Pad1.33x1.80mm_HandSolder -> Capacitor_SMD:C_1812_4532Metric_Pad1.57x3.40mm_HandSolder
- J1, J2: footprint (none) -> Connector_JST:JST_GH_BM04B-GHS-TBT_1x04-1MP_P1.25mm_Vertical
- R1: footprint Resistor_SMD:R_1206_3216Metric_Pad1.30x1.75mm_HandSolder -> Resistor_SMD:R_1812_4532Metric_Pad1.30x3.40mm_HandSolder
- R2: footprint (none) -> Resistor_SMD:R_1812_4532Metric_Pad1.30x3.40mm_HandSolder
- R3: value 120R -> 10kR
- R4: value 120R -> R
Connections:
- net GND: now also J3.2 (Pin_2), R3.2, C3.1, C3.2, C4.1, C4.2, C5.1, C5.2, C6.1, C6.2, C7.1, C7.2, C8.1, C8.2, C9.1, C9.2, CR5.1 (IO), CR5.2 (IO), CR6.1 (IO), CR6.2 (IO), D1.A, D1.K, D3.A, D3.K, D4.A, D4.K, D5.A, D5.K, D6.A, D6.K, D7.A, D7.K, J10.1 (Pin_1), J10.4 (Pin_4), J11.2 (Pin_2), J11.3 (Pin_3), J12.2 (Pin_2), J12.3 (Pin_3), J13.1 (Pin_1), J13.2 (Pin_2), J13.3 (Pin_3), J13.4 (Pin_4), J14.1 (Pin_1), J14.2 (Pin_2), J14.3 (Pin_3), J14.4 (Pin_4), J15.1 (Pin_1), J15.2 (Pin_2), J15.3 (Pin_3), J15.4 (Pin_4), J16.1 (Pin_1), J16.2 (Pin_2), J16.3 (Pin_3), J16.4 (Pin_4), J23.1 (Pin_1), J23.2 (Pin_2), J23.3 (Pin_3), J23.4 (Pin_4), J24.1 (Pin_1), J24.2 (Pin_2), J24.3 (Pin_3), J24.4 (Pin_4), J25.1 (Pin_1), J25.2 (Pin_2), J25.3 (Pin_3), J25.4 (Pin_4), J26.1 (Pin_1), J26.2 (Pin_2), J26.3 (Pin_3), J26.4 (Pin_4), J5.1 (Pin_1), J5.4 (Pin_4), J6.2 (Pin_2), J7.1 (Pin_1), J7.4 (Pin_4), J8.2 (Pin_2), J9.1 (Pin_1), J9.4 (Pin_4), R12.2, R14.2, R16.2, R18.1, R18.2, R19.2, R20.2, R21.2, R22.2, R23.2, R24.1, R25.1, R25.2, R29.1, R29.2, R30.1, R31.2, R32.2, R33.1, R34.1, R34.2, R7.2, SW3.1 (A), SW3.2 (A), SW6.3 (B), SW6.4 (B), U2.3 (GND), U2.4 (IN), U4.3 (GND), U4.4 (IN), U5.1 (COM), U5.3 (GND), U5.4 (IN), U6.1 (COM), U6.3 (GND), U6.4 (IN)
- net VCC 10V: now also J3.1 (Pin_1), J6.1 (Pin_1), J8.1 (Pin_1), R12.1, R19.1, R20.1, R22.1, R23.1, R31.1, R32.1, R7.1, U2.5 (V+), U4.5 (V+), U5.5 (V+), U6.5 (V+)
- net CAN_LOW: now reaches J4.1 (Pin_1)
- net CAN_LOW: now also J1.3 (Pin_3), J2.3 (Pin_3), R2.1, CR1.1 (IO), J17.1 (Pin_1), J18.2 (Pin_2)
- net CAN_HIGH: now reaches J4.2 (Pin_2)
- net CAN_HIGH: now also J1.2 (Pin_2), J2.2 (Pin_2), U1.1 (COM), CR1.2 (IO), J17.2 (Pin_2), J18.1 (Pin_1)
- new net: R17.1, U4.2 (NO)
- new net: CR3.2 (IO), CR4.2 (IO), J11.1 (Pin_1), J12.4 (Pin_4), R10.2, R11.2, R17.2, U2.1 (COM)
- new net: J5.2 (Pin_2), J7.2 (Pin_2), R4.1, R5.1, R9.1
- new net: J5.3 (Pin_3), J7.3 (Pin_3), R4.2, R5.2, R9.2, SW1.3 (B), SW1.4 (B)
- new net: R21.1, U5.2 (NO)
- new net: SW5.1 (A), SW5.2 (A)
- new net: SW5.3 (B), SW5.4 (B)
- new net: SW1.1 (A), SW1.2 (A)
- new net: R24.2, U6.2 (NO)
- new net: CR3.1 (IO), CR4.1 (IO), J11.4 (Pin_4), J12.1 (Pin_1), R10.1, R11.1, R8.1, U4.1 (COM)
- new net: J10.2 (Pin_2), J9.2 (Pin_2), R13.1, R15.1
- new net: J10.3 (Pin_3), J9.3 (Pin_3), R15.2, SW4.1 (A), SW4.2 (A)
- new net: R30.2, SW6.1 (A), SW6.2 (A)
- new net: R13.2, SW4.3 (B), SW4.4 (B)
- new net: R33.2, SW3.3 (B), SW3.4 (B)
- new net: R8.2, U2.2 (NO)
- new net GND_CAN: CR1.3 (GND), CR3.3 (GND), CR4.3 (GND), CR5.3 (GND), CR6.3 (GND)
- new net VCC: R14.1, R16.1, R3.1
Other:
- note added: "BLACK BOX"
- note added: "BOTTOM OF ROCKET CIRCUIT BOARD"
- note added: "C"
- note added: "GHOST RESISTOR"
- note added: "GHOST RESISTOR 120R"
- note added: "IN"
- note added: "JST CABLES (NOT PCB WIRING)"
- note added: "SPLIT RESISTOR"
- note added: "SPLT LINE"
- note added: "TOP OF ROCKET CIRCUIT BOARD"
- note added: "TVS"
- note added: "VERTICAL"
- moved on the sheet: C1, J2, J3, J4, R1, R2, U1
