File: CAN_BUS/CAN_BUS.kicad_sch (KiCad schematic)
At the start: 40 parts, among them J1 JST XH B2B-XH-A, J2 JST VH B2P-VH-FB-B, J23 Conn_01x04, J26 Conn_01x04, J3 Conn_01x04, J4 Conn_01x04, J5 JST VH B2P-VH-FB-B, J6 Conn_01x04, J7 JST XH B2B-XH-A, J8 JST VH B2P-VH-FB-B, J9 JST XH B2B-XH-A, SW3 SW_MEC_5G, SW6 SW_MEC_5G, U1 TS12A4514DBVR, U2 TS12A4514DBVR, U3 TS12A4514DBVR

Commit message: Add files via upload
Parts:
- removed C1, C2: 0.1uF, Capacitor_SMD:C_1812_4532Metric_Pad1.57x3.40mm_HandSolder, symbol Device:C
- removed CR1, CR2, CR3: ESD2CAN36DBZRQ1, SOT-23-3_DBZ_TEX, symbol ESD2CAN36-Q1:ESD2CAN36DBZRQ1
- removed D1, D2, D3: UCLAMP1071P.TNT, UCLAMP1071P.TNT:DIO_UCLAMP1071P.TNT, symbol UCLAMP1071P.TNT:UCLAMP1071P.TNT
- removed J1, J7, J9: JST XH B2B-XH-A, Connector_JST:JST_XH_B2B-XH-A_1x02_P2.50mm_Vertical, symbol Connector:Conn_01x02_Pin
- removed J2, J5, J8: JST VH B2P-VH-FB-B, Connector_JST:JST_VH_B2P-VH-FB-B_1x02_P3.96mm_Vertical, symbol Connector:Conn_01x02_Pin
- removed J23, J26, J3, J4, J6: Conn_01x04, Connector_JST:JST_GH_BM04B-GHS-TBT_1x04-1MP_P1.25mm_Vertical, symbol Connector_Generic:Conn_01x04
- removed R1, R2, R29, R30, R33, R34: 120R, symbol Device:R
- removed R3, R31, R32, R4: 10kR, Resistor_SMD:R_1812_4532Metric_Pad1.30x3.40mm_HandSolder, symbol Device:R
- removed R5, R6: 120R, Capacitor_SMD:C_1812_4532Metric_Pad1.57x3.40mm_HandSolder, symbol Device:R
- removed SW3, SW6: SW_MEC_5G, symbol Switch:SW_MEC_5G
- removed U1, U2, U3: TS12A4514DBVR, TS12A4514:DBV5, symbol TS12A4514:TS12A4514DBVR
- added C4: 0.1uF, Capacitor_SMD:C_0805_2012Metric_Pad1.18x1.45mm_HandSolder, symbol Device:C
- added C5: 10uF, Capacitor_SMD:C_0805_2012Metric_Pad1.18x1.45mm_HandSolder, symbol Device:C
- added CR4: ESD2CAN36DBZRQ1, SOT-23-3_DBZ_TEX, symbol ESD2CAN36-Q1:ESD2CAN36DBZRQ1
- added D4: UCLAMP1071P.TNT, UCLAMP1071P.TNT:DIO_UCLAMP1071P.TNT, symbol UCLAMP1071P.TNT:UCLAMP1071P.TNT
- added F1: 1.1A, Fuse:Fuse_1812_4532Metric_Pad1.30x3.40mm_HandSolder, symbol Device:Polyfuse
- added H3, H4, H5, H6: MountingHole_Pad, MountingHole:MountingHole_3.2mm_M3_Pad_Via, symbol Mechanical:MountingHole_Pad
- added J10, J19, J8, J9: Conn_01x04, Connector_JST:JST_GH_BM04B-GHS-TBT_1x04-1MP_P1.25mm_Vertical, symbol Connector_Generic:Conn_01x04
- added J11, J17, J6: JST_VH_IN/OUT, Connector_JST:JST_VH_B2P-VH-FB-B_1x02_P3.96mm_Vertical, symbol Connector:Conn_01x02_Pin
- added J16: JST_XH, Connector_JST:JST_XH_B2B-XH-A_1x02_P2.50mm_Vertical, symbol Connector:Conn_01x02_Pin
- added JST_XH_CAN1, JST_XH_SWITCH1: JST XH B2B-XH-A, Connector_JST:JST_XH_B2B-XH-A_1x02_P2.50mm_Vertical, symbol Connector:Conn_01x02_Pin
- added R10: 120R, Resistor_SMD:R_0805_2012Metric_Pad1.20x1.40mm_HandSolder, symbol Device:R
- added R11, R14: 1M, Resistor_SMD:R_0805_2012Metric_Pad1.20x1.40mm_HandSolder, symbol Device:R
- added U3: LM2937IMP-8.0, LM2937IMP-8.0:SOT230P700X180-4N, symbol LM2937IMP-8.0:LM2937IMP-8.0
- added U4: TS12A4514DBVR, TS12A4514:DBV5, symbol TS12A4514:TS12A4514DBVR
- C3: footprint Capacitor_SMD:C_1812_4532Metric_Pad1.57x3.40mm_HandSolder -> Capacitor_SMD:C_0805_2012Metric_Pad1.18x1.45mm_HandSolder
- R7: value 10kR -> 1M; footprint Resistor_SMD:R_1812_4532Metric_Pad1.30x3.40mm_HandSolder -> Resistor_SMD:R_0805_2012Metric_Pad1.20x1.40mm_HandSolder
- R8: value 120R -> 1M; footprint Capacitor_SMD:C_1812_4532Metric_Pad1.57x3.40mm_HandSolder -> Resistor_SMD:R_0805_2012Metric_Pad1.20x1.40mm_HandSolder
- R9: value 120R -> 10kR; footprint Capacitor_SMD:C_1812_4532Metric_Pad1.57x3.40mm_HandSolder -> Resistor_SMD:R_0805_2012Metric_Pad1.20x1.40mm_HandSolder
Connections:
- net CAN_HIGH: now also CR4.1 (IO), J10.3 (Pin_3), J16.1 (Pin_1), J19.3 (Pin_3), J8.3 (Pin_3), J9.3 (Pin_3), JST_XH_CAN1.2 (Pin_2), R10.1
- net CAN_LOW: now also CR4.2 (IO), J10.2 (Pin_2), J16.2 (Pin_2), J19.2 (Pin_2), J8.2 (Pin_2), J9.2 (Pin_2), JST_XH_CAN1.1 (Pin_1), U4.1 (COM)
- net GND: now also R7.2, R8.2, C4.1, C5.1, D4.K, J10.1 (Pin_1), J11.1 (Pin_1), J17.1 (Pin_1), J19.1 (Pin_1), J6.1 (Pin_1), J8.1 (Pin_1), J9.1 (Pin_1), JST_XH_SWITCH1.1 (Pin_1), R11.2, R14.2, U3.2 (GND), U4.3 (GND)
- net GND_CAN: now also CR4.3 (GND)
- net at C3.2: now also F1.1, U3.1 (VIN); no longer R7.2
- removed net SPLIT LINE: R8.1, R9.1, R9.2
- net VCC_10V: no longer names the net of R7.1
- net VCC_10V: now also H5.1
- new net: R10.2, U4.2 (NO)
- new net: H6.1, R14.1
- new net: H3.1, R11.1
- new net: H4.1, R8.1
- new net DW_POWER: F1.2, J11.2 (Pin_2), J17.2 (Pin_2), J6.2 (Pin_2)
- new net HEAT_SINK: U3.4 (GND_(TAB))
- new net SWITCH: C4.2, D4.A, JST_XH_SWITCH1.2 (Pin_2), R9.2, U4.4 (IN)
- new net VCC: J10.4 (Pin_4), J19.4 (Pin_4), J8.4 (Pin_4), J9.4 (Pin_4)
- new net V_REG: C5.2, R9.1, U3.3 (VOUT), U4.5 (V+)
Other:
- note added: "(DEDICATED INPUT)"
- note added: "8 VOLT OUTPUT"
- note added: "CAN GH SPLITTER OUTPUT + POWER"
- note added: "CAN ONLY"
- note removed: "BLACK BOX"
- note removed: "BOTTOM HALF"
- note removed: "BOTTOM OF ROCKET CIRCUIT BOARD"
- note removed: "CAN HIGH"
- note removed: "CAN LOW"
- note removed: "GHOST RESISTOR 120R"
- note removed: "IN"
- note removed: "TOP OF ROCKET CIRCUIT BOARD"
- note removed: "VERTICAL"
