File: CAN_BUS/CAN_BUS.kicad_pcb (KiCad board)
At the start: 2 copper layers, 14 x 5.5 mm, 0 parts

Commit message: Add files via upload
Other:
- board outline removed
Changed lines of the file:
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@@
 	)
 	(net 0 "")
-	(gr_rect
-		(start 143 74.5)
-		(end 157 80)
-		(stroke
-			(width 0.05)
-			(type default)
-		)
-		(fill none)
-		(layer "Edge.Cuts")
-	)
 )

Commit message: Add files via upload
Parts:
- added C3: 0.1uF, Capacitor_SMD:C_0805_2012Metric_Pad1.18x1.45mm_HandSolder, F.Cu at (139.8, 81.3)
- added C4: 0.1uF, Capacitor_SMD:C_0805_2012Metric_Pad1.18x1.45mm_HandSolder, F.Cu at (139.8, 84.3)
- added C5: 10uF, Capacitor_SMD:C_0805_2012Metric_Pad1.18x1.45mm_HandSolder, F.Cu at (139.8, 87.3)
- added CR4: ESD2CAN36DBZRQ1, ESD2CAN36-Q1:SOT-23-3_DBZ_TEX, F.Cu at (105.4, 94.1)
- added D4: UCLAMP1071P.TNT, UCLAMP1071P.TNT:DIO_UCLAMP1071P.TNT, F.Cu at (126.9, 94.4)
- added F1: 1.1A, Fuse:Fuse_1812_4532Metric_Pad1.30x3.40mm_HandSolder, F.Cu at (128.3, 90.7)
- added H3: MountingHole_Pad, MountingHole:MountingHole_3.2mm_M3_Pad_Via, F.Cu at (128.7, 60.4)
- added H4: MountingHole_Pad, MountingHole:MountingHole_3.2mm_M3_Pad_Via, F.Cu at (128.7, 68.3)
- added H5: MountingHole_Pad, MountingHole:MountingHole_3.2mm_M3_Pad_Via, F.Cu at (128.7, 76.2)
- added H6: MountingHole_Pad, MountingHole:MountingHole_3.2mm_M3_Pad_Via, F.Cu at (128.7, 84.2)
- added J10: Conn_01x04, Connector_JST:JST_GH_BM04B-GHS-TBT_1x04-1MP_P1.25mm_Vertical, F.Cu at (119.4, 75.5)
- added J11: JST_VH_IN/OUT, Connector_JST:JST_VH_B2P-VH-FB-B_1x02_P3.96mm_Vertical, F.Cu at (106.3, 73.7)
- added J16: JST_XH, Connector_JST:JST_XH_B2B-XH-A_1x02_P2.50mm_Vertical, F.Cu at (136.1, 59.8)
- added J17: JST_VH_IN/OUT, Connector_JST:JST_VH_B2P-VH-FB-B_1x02_P3.96mm_Vertical, F.Cu at (106.3, 85.4)
- added J19: Conn_01x04, Connector_JST:JST_GH_BM04B-GHS-TBT_1x04-1MP_P1.25mm_Vertical, F.Cu at (119.4, 83.2)
- added J6: JST_VH_IN/OUT, Connector_JST:JST_VH_B2P-VH-FB-B_1x02_P3.96mm_Vertical, F.Cu at (106.3, 61.9)
- added J8: Conn_01x04, Connector_JST:JST_GH_BM04B-GHS-TBT_1x04-1MP_P1.25mm_Vertical, F.Cu at (119.4, 60.2)
- added J9: Conn_01x04, Connector_JST:JST_GH_BM04B-GHS-TBT_1x04-1MP_P1.25mm_Vertical, F.Cu at (119.4, 67.8)
- added JST_XH_CAN1: JST XH B2B-XH-A, Connector_JST:JST_XH_B2B-XH-A_1x02_P2.50mm_Vertical, F.Cu at (136.1, 67.5)
- added JST_XH_SWITCH1: JST XH B2B-XH-A, Connector_JST:JST_XH_B2B-XH-A_1x02_P2.50mm_Vertical, F.Cu at (136.1, 75.3)
- added R10: 120R, Resistor_SMD:R_0805_2012Metric_Pad1.20x1.40mm_HandSolder, F.Cu at (135.0, 90.1)
- added R11: 1M, Resistor_SMD:R_0805_2012Metric_Pad1.20x1.40mm_HandSolder, F.Cu at (135.0, 93.0)
- added R14: 1M, Resistor_SMD:R_0805_2012Metric_Pad1.20x1.40mm_HandSolder, F.Cu at (135.0, 96.0)
- added R7: 1M, Resistor_SMD:R_0805_2012Metric_Pad1.20x1.40mm_HandSolder, F.Cu at (135.0, 81.2)
- added R8: 1M, Resistor_SMD:R_0805_2012Metric_Pad1.20x1.40mm_HandSolder, F.Cu at (135.0, 84.2)
- added R9: 10kR, Resistor_SMD:R_0805_2012Metric_Pad1.20x1.40mm_HandSolder, F.Cu at (135.0, 87.2)
- added U3: LM2937IMP-8.0, LM2937IMP-8.0:SOT230P700X180-4N, F.Cu at (119.5, 91.0)
- added U4: TS12A4514DBVR, TS12A4514:DBV5, F.Cu at (110.5, 94.0)
